Commit message: ros integration

File: assets/g1/g1_29dof_with_hand_rev_1_0_ros.urdf (robot description, URDF)
Before this commit: robot g1_29dof_with_hand_rev_1_0, 54 links, 53 joints
Links:
- removed link base
- added link g1_center
- link head_link: geometry collision mesh filename=package://g1_ik/assets/g1/meshes/head_link.STL; visual mesh filename=package://g1_ik/assets/g1/meshes/head_link.STL
- link left_ankle_pitch_link: geometry collision mesh filename=package://g1_ik/assets/g1/meshes/left_ankle_pitch_link.STL; visual mesh filename=package://g1_ik/assets/g1/meshes/left_ankle_pitch_link.STL
- link left_ankle_roll_link: geometry collision sphere radius=0.005; collision sphere radius=0.005
- link left_elbow_link: geometry collision mesh filename=package://g1_ik/assets/g1/meshes/left_elbow_link.STL; visual mesh filename=package://g1_ik/assets/g1/meshes/left_elbow_link.STL
- link left_hand_index_0_link: geometry collision mesh filename=package://g1_ik/assets/g1/meshes/left_hand_index_0_link.STL; visual mesh filename=package://g1_ik/assets/g1/meshes/left_hand_index_0_link.STL
- link left_hand_index_1_link: geometry collision mesh filename=package://g1_ik/assets/g1/meshes/left_hand_index_1_link.STL; visual mesh filename=package://g1_ik/assets/g1/meshes/left_hand_index_1_link.STL
- link left_hand_middle_0_link: geometry collision mesh filename=package://g1_ik/assets/g1/meshes/left_hand_middle_0_link.STL; visual mesh filename=package://g1_ik/assets/g1/meshes/left_hand_middle_0_link.STL
- link left_hand_middle_1_link: geometry collision mesh filename=package://g1_ik/assets/g1/meshes/left_hand_middle_1_link.STL; visual mesh filename=package://g1_ik/assets/g1/meshes/left_hand_middle_1_link.STL
- link left_hand_palm_link: geometry collision mesh filename=package://g1_ik/assets/g1/meshes/left_hand_palm_link.STL; visual mesh filename=package://g1_ik/assets/g1/meshes/left_hand_palm_link.STL
- link left_hand_thumb_0_link: geometry collision mesh filename=package://g1_ik/assets/g1/meshes/left_hand_thumb_0_link.STL; visual mesh filename=package://g1_ik/assets/g1/meshes/left_hand_thumb_0_link.STL
- link left_hand_thumb_1_link: geometry collision box size=0.02 0.03 0.02; visual mesh filename=package://g1_ik/assets/g1/meshes/left_hand_thumb_1_link.STL
- link left_hand_thumb_2_link: geometry collision mesh filename=package://g1_ik/assets/g1/meshes/left_hand_thumb_2_link.STL; visual mesh filename=package://g1_ik/assets/g1/meshes/left_hand_thumb_2_link.STL
- link left_hip_pitch_link: geometry collision mesh filename=package://g1_ik/assets/g1/meshes/left_hip_pitch_link.STL; visual mesh filename=package://g1_ik/assets/g1/meshes/left_hip_pitch_link.STL
- link left_hip_roll_link: geometry collision mesh filename=package://g1_ik/assets/g1/meshes/left_hip_roll_link.STL; visual mesh filename=package://g1_ik/assets/g1/meshes/left_hip_roll_link.STL
- link left_hip_yaw_link: geometry collision mesh filename=package://g1_ik/assets/g1/meshes/left_hip_yaw_link.STL; visual mesh filename=package://g1_ik/assets/g1/meshes/left_hip_yaw_link.STL
- link left_knee_link: geometry collision mesh filename=package://g1_ik/assets/g1/meshes/left_knee_link.STL; visual mesh filename=package://g1_ik/assets/g1/meshes/left_knee_link.STL
- link left_shoulder_pitch_link: geometry collision cylinder length=0.05 radius=0.03; visual mesh filename=package://g1_ik/assets/g1/meshes/left_shoulder_pitch_link.S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
- link left_shoulder_roll_link: geometry collision cylinder length=0.03 radius=0.03; visual mesh filename=package://g1_ik/assets/g1/meshes/left_shoulder_roll_link.STL
- link left_shoulder_yaw_link: geometry collision mesh filename=package://g1_ik/assets/g1/meshes/left_shoulder_yaw_link.STL; visual mesh filename=package://g1_ik/assets/g1/meshes/left_shoulder_yaw_link.STL
- link left_wrist_pitch_link: geometry collision mesh filename=package://g1_ik/assets/g1/meshes/left_wrist_pitch_link.STL; visual mesh filename=package://g1_ik/assets/g1/meshes/left_wrist_pitch_link.STL
- link left_wrist_roll_link: geometry collision mesh filename=package://g1_ik/assets/g1/meshes/left_wrist_roll_link.STL; visual mesh filename=package://g1_ik/assets/g1/meshes/left_wrist_roll_link.STL
- link left_wrist_yaw_link: geometry collision mesh filename=package://g1_ik/assets/g1/meshes/left_wrist_yaw_link.STL; visual mesh filename=package://g1_ik/assets/g1/meshes/left_wrist_yaw_link.STL
- link logo_link: geometry collision mesh filename=package://g1_ik/assets/g1/meshes/logo_link.STL; visual mesh filename=package://g1_ik/assets/g1/meshes/logo_link.STL
- link pelvis: geometry visual mesh filename=package://g1_ik/assets/g1/meshes/pelvis.STL
- link pelvis_contour_link: geometry collision mesh filename=package://g1_ik/assets/g1/meshes/pelvis_contour_link.STL; visual mesh filename=package://g1_ik/assets/g1/meshes/pelvis_contour_link.STL
- link right_ankle_pitch_link: geometry collision mesh filename=package://g1_ik/assets/g1/meshes/right_ankle_pitch_link.STL; visual mesh filename=package://g1_ik/assets/g1/meshes/right_ankle_pitch_link.STL
- link right_ankle_roll_link: geometry collision sphere radius=0.005; collision sphere radius=0.005
- link right_elbow_link: geometry collision mesh filename=package://g1_ik/assets/g1/meshes/right_elbow_link.STL; visual mesh filename=package://g1_ik/assets/g1/meshes/right_elbow_link.STL
- link right_hand_index_0_link: geometry collision mesh filename=package://g1_ik/assets/g1/meshes/right_hand_index_0_link.STL; visual mesh filename=package://g1_ik/assets/g1/meshes/right_hand_index_0_link.STL
- link right_hand_index_1_link: geometry collision mesh filename=package://g1_ik/assets/g1/meshes/right_hand_index_1_link.STL; visual mesh filename=package://g1_ik/assets/g1/meshes/right_hand_index_1_link.STL
- link right_hand_middle_0_link: geometry collision mesh filename=package://g1_ik/assets/g1/meshes/right_hand_middle_0_link.S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; visual mesh filename=package://g1_ik/assets/g1/meshes/right_hand_middle_0_link.S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
- link right_hand_middle_1_link: geometry collision mesh filename=package://g1_ik/assets/g1/meshes/right_hand_middle_1_link.S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; visual mesh filename=package://g1_ik/assets/g1/meshes/right_hand_middle_1_link.S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
- link right_hand_palm_link: geometry collision mesh filename=package://g1_ik/assets/g1/meshes/right_hand_palm_link.STL; visual mesh filename=package://g1_ik/assets/g1/meshes/right_hand_palm_link.STL
- link right_hand_thumb_0_link: geometry collision mesh filename=package://g1_ik/assets/g1/meshes/right_hand_thumb_0_link.STL; visual mesh filename=package://g1_ik/assets/g1/meshes/right_hand_thumb_0_link.STL
- link right_hand_thumb_1_link: geometry collision box size=0.02 0.03 0.02; visual mesh filename=package://g1_ik/assets/g1/meshes/right_hand_thumb_1_link.STL
- link right_hand_thumb_2_link: geometry collision mesh filename=package://g1_ik/assets/g1/meshes/right_hand_thumb_2_link.STL; visual mesh filename=package://g1_ik/assets/g1/meshes/right_hand_thumb_2_link.STL
- link right_hip_pitch_link: geometry collision mesh filename=package://g1_ik/assets/g1/meshes/right_hip_pitch_link.STL; visual mesh filename=package://g1_ik/assets/g1/meshes/right_hip_pitch_link.STL
- link right_hip_roll_link: geometry collision mesh filename=package://g1_ik/assets/g1/meshes/right_hip_roll_link.STL; visual mesh filename=package://g1_ik/assets/g1/meshes/right_hip_roll_link.STL
- link right_hip_yaw_link: geometry collision mesh filename=package://g1_ik/assets/g1/meshes/right_hip_yaw_link.STL; visual mesh filename=package://g1_ik/assets/g1/meshes/right_hip_yaw_link.STL
- link right_knee_link: geometry collision mesh filename=package://g1_ik/assets/g1/meshes/right_knee_link.STL; visual mesh filename=package://g1_ik/assets/g1/meshes/right_knee_link.STL
- link right_shoulder_pitch_link: geometry collision cylinder length=0.05 radius=0.03; visual mesh filename=package://g1_ik/assets/g1/meshes/right_shoulder_pitch_link.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
- link right_shoulder_roll_link: geometry collision cylinder length=0.03 radius=0.03; visual mesh filename=package://g1_ik/assets/g1/meshes/right_shoulder_roll_link.S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
- link right_shoulder_yaw_link: geometry collision mesh filename=package://g1_ik/assets/g1/meshes/right_shoulder_yaw_link.STL; visual mesh filename=package://g1_ik/assets/g1/meshes/right_shoulder_yaw_link.STL
- link right_wrist_pitch_link: geometry collision mesh filename=package://g1_ik/assets/g1/meshes/right_wrist_pitch_link.STL; visual mesh filename=package://g1_ik/assets/g1/meshes/right_wrist_pitch_link.STL
- link right_wrist_roll_link: geometry collision mesh filename=package://g1_ik/assets/g1/meshes/right_wrist_roll_link.STL; visual mesh filename=package://g1_ik/assets/g1/meshes/right_wrist_roll_link.STL
- link right_wrist_yaw_link: geometry collision mesh filename=package://g1_ik/assets/g1/meshes/right_wrist_yaw_link.STL; visual mesh filename=package://g1_ik/assets/g1/meshes/right_wrist_yaw_link.STL
- link torso_link: geometry collision mesh filename=package://g1_ik/assets/g1/meshes/torso_link_rev_1_0.STL; visual mesh filename=package://g1_ik/assets/g1/meshes/torso_link_rev_1_0.STL
- link waist_roll_link: geometry visual mesh filename=package://g1_ik/assets/g1/meshes/waist_roll_link_rev_1_0.STL
- link waist_yaw_link: geometry visual mesh filename=package://g1_ik/assets/g1/meshes/waist_yaw_link_rev_1_0.STL
Joints:
- joint g1_reference_to_pelvis_joint: parent base -> g1_center
